Commit message: Updated URDF to be upright

File: robots/scrap_arm.urdf (robot description, URDF)
Before this commit: robot scrap_arm, 3 links, 2 joints
Links:
- link Link00: mass 0.041843 -> None
- link Link01: mass 0.054343 -> None
- link base_link: mass 7.0765 -> None
Joints:
- joint Joint00: origin xyz=0 -0.13 0 rpy=1.5708 0 3.1416 -> xyz=0 0 0.13 rpy=0 3.14159625 0
