Commit message: Moved STLs to URDF

File: urdf/scrap_arm.urdf (robot description, URDF)
Before this commit: robot scrap_arm, 3 links, 2 joints
Links:
- link Link00: geometry collision mesh filename=package://scrap_arm/urdf/Link00.STL; visual mesh filename=package://scrap_arm/urdf/Link00.STL
- link Link01: geometry collision mesh filename=package://scrap_arm/urdf/Link01.STL; visual mesh filename=package://scrap_arm/urdf/Link01.STL
- link base_link: geometry collision mesh filename=package://scrap_arm/urdf/base_link.STL; visual mesh filename=package://scrap_arm/urdf/base_link.STL
